File: 8ch_mas_flex.kicad_pcb (KiCad board)
At the start: 2 copper layers, 567.6 x 101.6 mm, 3 parts, among them J1 2-5174225-5, U1 QIS_SKCCD_8CH_inline-qis

Commit message: updated kicad version?
Parts:
- moved U1 20.0 mm to (-108.4, 97.9)
Routing:
- net VOUT-U2: track 565.8 -> 545.8 mm
- net VDD: track 576.2 -> 556.2 mm
- net SW-B: track 550.9 -> 530.9 mm
- net OG-A: track 556.8 -> 536.8 mm
- net H3-A: track 571.0 -> 551.0 mm
- net H1-B: track 552.1 -> 532.1 mm
- net VOUT-U2-CCD: track 559.3 -> 539.3 mm
- net VOUT-U1: track 590.9 -> 570.9 mm
- net VOUT-L2: track 547.4 -> 527.4 mm
- net RG-B: track 548.6 -> 528.6 mm
- net RG-A: track 541.6 -> 521.6 mm
- net RD-L2: track 543.8 -> 523.8 mm
- net OG-B: track 546.1 -> 526.1 mm
- net H3-B: track 548.6 -> 528.6 mm
- net H2: track 567.6 -> 547.6 mm
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- added copper zone on B.Cu, net BIAS_GRD
Other:
- outline, holes or cut-outs redrawn
- board text added: "Flex for 8-CH MAS-CCD 08–Aug-2022 v1.1"
- board text removed: "Flex for 8-CH MAS-CCD 04–May-2022"
